Commit message: urdf modif

File: src/asterix/robot/asterix.urdf (robot description, URDF)
Before this commit: robot Asterix, 4 links, 3 joints
Joints:
- joint base_joint: origin xyz=0.0 0.0 0.5 rpy=0 0 0 -> xyz=0.0 0.0 0.0 rpy=0 0 0

Commit message: urdf bien

File: src/asterix/robot/asterix.urdf (robot description, URDF)
Before this commit: robot Asterix, 4 links, 3 joints
Joints:
- joint wheel_left_joint: axis 1 0 0 -> 0 1 0; origin xyz=0.0 0.08 0.023 rpy=-1.57 0 0 -> xyz=0.0 0.08 0.023 rpy=0 0 0
- joint wheel_right_joint: axis 1 0 0 -> 0 1 0; origin xyz=0.0 -0.080 0.023 rpy=-1.57 0 0 -> xyz=0.0 -0.080 0.023 rpy=0 0 0

Commit message: Urdf bien avec les cotes

File: src/asterix/robot/asterix.urdf (robot description, URDF)
Before this commit: robot Asterix, 4 links, 3 joints
Links:
- link robotbase: geometry collision box size=0.25 0.30 0.35; visual box size=0.2 0.26 0.32
- link wheel_left_link: geometry visual cylinder length=0.01 radius=0.04
- link wheel_right_link: geometry visual cylinder length=0.01 radius=0.04
Joints:
- joint base_joint: origin xyz=0.0 0.0 0.0 rpy=0 0 0 -> xyz=0.0 0.0 0.16 rpy=0 0 0
- joint wheel_left_joint: origin xyz=0.0 0.08 0.023 rpy=0 0 0 -> xyz=0.0 0.13 -0.13 rpy=0 0 0
- joint wheel_right_joint: origin xyz=0.0 -0.080 0.023 rpy=0 0 0 -> xyz=0.0 -0.13 -0.13 rpy=0 0 0

Commit message: URDF

File: src/asterix/robot/asterix.urdf (robot description, URDF)
Before this commit: robot Asterix, 4 links, 3 joints
Links:
- link robotbase: geometry collision box size=0.140 0.140 0.143; visual box size=0.140 0.140 0.143
- link wheel_left_link: geometry collision cylinder length=0.018 radius=0.033; visual cylinder length=0.018 radius=0.033
- link wheel_right_link: geometry collision cylinder length=0.018 radius=0.033; visual cylinder length=0.018 radius=0.033
Joints:
- joint base_joint: origin xyz=0.0 0.0 0.16 rpy=0 0 0 -> xyz=0.0 0.0 0.5 rpy=0 0 0
- joint wheel_left_joint: axis 0 1 0 -> 1 0 0; origin xyz=0.0 0.13 -0.13 rpy=0 0 0 -> xyz=0.0 0.08 0.023 rpy=-1.57 0 0
- joint wheel_right_joint: axis 0 1 0 -> 1 0 0; origin xyz=0.0 -0.13 -0.13 rpy=0 0 0 -> xyz=0.0 -0.080 0.023 rpy=-1.57 0 0

Commit message: Correct URDF

File: src/asterix/robot/asterix.urdf (robot description, URDF)
Before this commit: robot Asterix, 4 links, 3 joints
Links:
- link robotbase: geometry collision box size=0.25 0.30 0.35; visual box size=0.2 0.26 0.32
- link wheel_left_link: geometry visual cylinder length=0.01 radius=0.04
- link wheel_right_link: geometry visual cylinder length=0.01 radius=0.04
Joints:
- joint base_joint: origin xyz=0.0 0.0 0.5 rpy=0 0 0 -> xyz=0.0 0.0 0.16 rpy=0 0 0
- joint wheel_left_joint: axis 1 0 0 -> 0 1 0; origin xyz=0.0 0.08 0.023 rpy=-1.57 0 0 -> xyz=0.0 0.13 -0.13 rpy=0 0 0
- joint wheel_right_joint: axis 1 0 0 -> 0 1 0; origin xyz=0.0 -0.080 0.023 rpy=-1.57 0 0 -> xyz=0.0 -0.13 -0.13 rpy=0 0 0

Commit message: base_footprint -> base_link

File: src/asterix/robot/asterix.urdf (robot description, URDF)
Before this commit: robot Asterix, 4 links, 3 joints
Links:
- removed link base_footprint
- added link base_link
Joints:
- joint base_joint: parent base_footprint -> base_link

Commit message: URDF Sensors

File: src/asterix/robot/asterix.urdf (robot description, URDF)
Before this commit: robot Asterix, 8 links, 3 joints
Links:
- link sensor_back_left: geometry visual box size=0.02 0.05 0.02
- link sensor_back_right: geometry visual box size=0.02 0.05 0.02
- link sensor_front_left: geometry visual box size=0.02 0.05 0.02
- link sensor_front_right: geometry visual box size=0.02 0.05 0.02
Joints:
- added joint sensor_back_left_joint: type fixed, parent robotbase, child sensor_back_left, origin xyz=-0.1 0.1 0.05 rpy=0 0 0
- added joint sensor_back_right_joint: type fixed, parent robotbase, child sensor_back_right, origin xyz=-0.1 -0.1 0.05 rpy=0 0 0
- added joint sensor_front_left_joint: type fixed, parent robotbase, child sensor_front_left, origin xyz=0.1 0.1 0.05 rpy=0 0 0
- added joint sensor_front_right_joint: type fixed, parent robotbase, child sensor_front_right, origin xyz=0.1 -0.1 0.05 rpy=0 0 0

Commit message: Updated sensors graphics

File: src/asterix/robot/asterix.urdf (robot description, URDF)
Before this commit: robot Asterix, 8 links, 7 joints
Links:
- link sensor_back_left: geometry visual box size=0.01 0.05 0.02
- link sensor_back_right: geometry visual box size=0.01 0.05 0.02
- link sensor_front_left: geometry visual box size=0.01 0.05 0.02
- link sensor_front_right: geometry visual box size=0.01 0.05 0.02
Joints:
- joint sensor_back_left_joint: origin xyz=-0.1 0.1 0.05 rpy=0 0 0 -> xyz=-0.096 0.1 0.05 rpy=0 0 0
- joint sensor_back_right_joint: origin xyz=-0.1 -0.1 0.05 rpy=0 0 0 -> xyz=-0.096 -0.1 0.05 rpy=0 0 0
- joint sensor_front_left_joint: origin xyz=0.1 0.1 0.05 rpy=0 0 0 -> xyz=0.096 0.1 0.05 rpy=0 0 0
- joint sensor_front_right_joint: origin xyz=0.1 -0.1 0.05 rpy=0 0 0 -> xyz=0.096 -0.1 0.05 rpy=0 0 0

Commit message: URDF retourner

File: src/asterix/robot/asterix.urdf (robot description, URDF)
Before this commit: robot Asterix, 8 links, 7 joints
Joints:
- joint sensor_back_left_joint: origin xyz=-0.096 0.1 0.05 rpy=0 0 0 -> xyz=-0.096 0.1 0.05 rpy=0 0 1,57
- joint sensor_back_right_joint: origin xyz=-0.096 -0.1 0.05 rpy=0 0 0 -> xyz=-0.096 -0.1 0.05 rpy=0 0 1,57
