Commit message: Sensors is now a macro

File: tools/xacro/robot.xacro (robot description, xacro)
@@ -4,4 +4,5 @@
   <xacro:include filename="colors.xacro"/>
   <xacro:include filename="inertias.xacro"/>
+  <xacro:include filename="sensors.xacro"/>
   <link name="$(arg tf_prefix)base_link"/>
   <joint name="$(arg tf_prefix)base_joint" type="fixed">
@@ -60,58 +61,8 @@
     </visual>
   </link>
-  <joint name="$(arg tf_prefix)sensor_front_left_joint" type="fixed">
-    <parent link="$(arg tf_prefix)robotbase"/>
-    <child link="$(arg tf_prefix)sensor_front_left"/>
-    <origin xyz="0.096 0.1 0.05" rpy="0 0 0"/>
-  </joint>
-  <link name="$(arg tf_prefix)sensor_front_left">
-    <visual>
-      <origin xyz="0 0 0" rpy="0 0 0"/>
-      <geometry>
-        <box size="0.01 0.05 0.02"/>
-      </geometry>
-      <material name="white"/>
-    </visual>
-  </link>
-  <joint name="$(arg tf_prefix)sensor_front_right_joint" type="fixed">
-    <parent link="$(arg tf_prefix)robotbase"/>
-    <child link="$(arg tf_prefix)sensor_front_right"/>
-    <origin xyz="0.096 -0.1 0.05" rpy="0 0 0"/>
-  </joint>
-  <link name="$(arg tf_prefix)sensor_front_right">
-    <visual>
-      <origin xyz="0 0 0" rpy="0 0 0"/>
-      <geometry>
-        <box size="0.01 0.05 0.02"/>
-      </geometry>
-      <material name="white"/>
-    </visual>
-  </link>
-  <joint name="$(arg tf_prefix)sensor_back_left_joint" type="fixed">
-    <parent link="$(arg tf_prefix)robotbase"/>
-    <child link="$(arg tf_prefix)sensor_back_left"/>
-  </joint>
-  <link name="$(arg tf_prefix)sensor_back_left">
-    <visual>
-      <origin xyz="0 0 0" rpy="0 0 0"/>
-      <geometry>
-        <box size="0.01 0.05 0.02"/>
-      </geometry>
-      <material name="white"/>
-    </visual>
-  </link>
-  <joint name="$(arg tf_prefix)sensor_back_right_joint" type="fixed">
-    <parent link="$(arg tf_prefix)robotbase"/>
-    <child link="$(arg tf_prefix)sensor_back_right"/>
-    <origin xyz="-0.096 -0.1 0.05" rpy="0 0 3.14159"/>
-  </joint>
-  <link name="$(arg tf_prefix)sensor_back_right">
-    <visual>
-      <origin xyz="0 0 0" rpy="0 0 0"/>
-      <geometry>
-        <box size="0.01 0.05 0.02"/>
-      </geometry>
-      <material name="white"/>
-    </visual>
-  </link>
+  <!--Sensors-->
+  <xacro:hcsr04_sensor name="sensor_front_left" xyz="0.096 0.1 0.05" rpy="0 0 0"/>
+  <xacro:hcsr04_sensor name="sensor_front_right" xyz="0.096 -0.1 0.05" rpy="0 0 0"/>
+  <xacro:hcsr04_sensor name="sensor_back_left" xyz="-0.096 0.1 0.05" rpy="0 0 0"/>
+  <xacro:hcsr04_sensor name="sensor_back_right" xyz="-0.096 -0.1 0.05" rpy="0 0 0"/>
 </robot>

Commit message: Updated prefix

File: tools/xacro/robot.xacro (robot description, xacro)
@@ -1,14 +1,14 @@
 <?xml version="1.0" ?>
 <robot name="${robot}" xmlns:xacro="http://www.ros.org/wiki/xacro">
-  <xacro:arg name="tf_prefix" default="${robot}/"/>
+  <xacro:property name="tf_prefix" value="${robot}/"/>
   <xacro:include filename="colors.xacro"/>
   <xacro:include filename="inertias.xacro"/>
-  <link name="$(arg tf_prefix)base_link"/>
-  <joint name="$(arg tf_prefix)base_joint" type="fixed">
-    <parent link="$(arg tf_prefix)base_link"/>
-    <child link="$(arg tf_prefix)robotbase"/>
+  <link name="${tf_prefix}base_link"/>
+  <joint name="${tf_prefix}base_joint" type="fixed">
+    <parent link="${tf_prefix}base_link"/>
+    <child link="${tf_prefix}robotbase"/>
     <origin xyz="0.0 0.0 0.16" rpy="0 0 0"/>
   </joint>
-  <link name="$(arg tf_prefix)robotbase">
+  <link name="${tf_prefix}robotbase">
     <xacro:box_inertia m="4" w="${robotbase_lenght}" h="${robotbase_width}" d="${robotbase_height}"/>
     <visual>
@@ -26,13 +26,13 @@
     </collision>
   </link>
-  <joint name="$(arg tf_prefix)wheel_left_joint" type="continuous">
-    <parent link="$(arg tf_prefix)robotbase"/>
-    <child link="$(arg tf_prefix)wheel_left_link"/>
+  <joint name="${tf_prefix}wheel_left_joint" type="continuous">
+    <parent link="${tf_prefix}robotbase"/>
+    <child link="${tf_prefix}wheel_left_link"/>
     <origin xyz="0.0 ${robotbase_width/2} -${robotbase_width/2}" rpy="0 0 0"/>
     <axis xyz="0 1 0"/>
     <dynamics damping="0.7"/>
   </joint>
-  <link name="$(arg tf_prefix)wheel_left_link">
-    <xacro:cylinder_inertia m="0.2" r="0.04" h="0.01"/>
+  <link name="${tf_prefix}wheel_left_link">
+    <xacro:cylinder_inertia m="0.2" r="${wheel_radius}" h="${wheel_width}"/>
     <visual>
       <origin xyz="0 0 0" rpy="1.57 0 0"/>
@@ -43,13 +43,13 @@
     </visual>
   </link>
-  <joint name="$(arg tf_prefix)wheel_right_joint" type="continuous">
-    <parent link="$(arg tf_prefix)robotbase"/>
-    <child link="$(arg tf_prefix)wheel_right_link"/>
+  <joint name="${tf_prefix}wheel_right_joint" type="continuous">
+    <parent link="${tf_prefix}robotbase"/>
+    <child link="${tf_prefix}wheel_right_link"/>
     <origin xyz="0.0 -${robotbase_width/2} -${robotbase_width/2}" rpy="0 0 0"/>
     <axis xyz="0 1 0"/>
     <dynamics damping="0.7"/>
   </joint>
-  <link name="$(arg tf_prefix)wheel_right_link">
-    <xacro:cylinder_inertia m="0.2" r="0.04" h="0.01"/>
+  <link name="${tf_prefix}wheel_right_link">
+    <xacro:cylinder_inertia m="0.2" r="${wheel_radius}" h="${wheel_width}"/>
     <visual>
       <origin xyz="0 0 0" rpy="1.57 0 0"/>
