Commit message: Updated URDF and xacro tool

File: tools/xacro/asterix.xacro (robot description, xacro)
@@ -1,54 +1,6 @@
 <?xml version="1.0" ?>
-<robot name="Asterix" xmlns:xacro="http://www.ros.org/wiki/xacro">
+<robot name="asterix" xmlns:xacro="http://www.ros.org/wiki/xacro">
   <xacro:include filename="colors.xacro"/>
-  <material name="black">
-      <color rgba="0.0 0.0 0.0 1.0"/>
-  </material>
-  <material name="dark">
-    <color rgba="0.3 0.3 0.3 1.0"/>
-  </material>
-  <material name="light_black">
-    <color rgba="0.4 0.4 0.4 1.0"/>
-  </material>
-  <material name="blue">
-    <color rgba="0.0 0.0 0.8 1.0"/>
-  </material>
-  <material name="green">
-    <color rgba="0.0 0.8 0.0 1.0"/>
-  </material>
-  <material name="grey">
-    <color rgba="0.5 0.5 0.5 1.0"/>
-  </material>
-  <material name="orange">
-    <color rgba="1.0 0.4235 0.0392 1.0"/>
-  </material>
-  <material name="brown">
-    <color rgba="0.8706 0.8118 0.7647 1.0"/>
-  </material>
-  <material name="red">
-    <color rgba="0.8 0.0 0.0 1.0"/>
-  </material>
-  <material name="white">
-    <color rgba="1.0 1.0 1.0 1.0"/>
-  </material>
-  <!--Interial macros-->
-  <xacro:macro name="cylinder_inertia" params="m r h">
-    <inertial>
-      <mass value="${m}"/>
-      <inertia ixx="${m*(3*r*r+h*h)/12}" ixy = "0" ixz = "0" iyy="${m*(3*r*r+h*h)/12}" iyz = "0" izz="${m*r*r/2}"/>
-    </inertial>
-  </xacro:macro>
-  <xacro:macro name="box_inertia" params="m w h d">
-    <inertial>
-      <mass value="${m}"/>
-      <inertia ixx="${m / 12.0 * (d*d + h*h)}" ixy="0.0" ixz="0.0" iyy="${m / 12.0 * (w*w + h*h)}" iyz="0.0" izz="${m / 12.0 * (w*w + d*d)}"/>
-    </inertial>
-  </xacro:macro>
-  <xacro:macro name="sphere_inertia" params="m r">
-    <inertial>
-      <mass value="${m}"/>
-      <inertia ixx="${2.0*m*(r*r)/5.0}" ixy="0.0" ixz="0.0" iyy="${2.0*m*(r*r)/5.0}" iyz="0.0" izz="${2.0*m*(r*r)/5.0}"/>
-    </inertial>
-  </xacro:macro>
+  <xacro:include filename="inertias.xacro"/>
   <link name="base_link"/>
   <joint name="base_joint" type="fixed">
@@ -138,5 +90,5 @@
     <parent link="robotbase"/>
     <child link="sensor_back_left"/>
-    <origin xyz="-0.096 0.1 0.05" rpy="0 0 1,57"/>
+    <origin xyz="-0.096 0.1 0.05" rpy="0 0 1.57"/>
   </joint>
   <link name="sensor_back_left">
@@ -152,5 +104,5 @@
     <parent link="robotbase"/>
     <child link="sensor_back_right"/>
-    <origin xyz="-0.096 -0.1 0.05" rpy="0 0 1,57"/>
+    <origin xyz="-0.096 -0.1 0.05" rpy="0 0 1.57"/>
   </joint>
   <link name="sensor_back_right">

Commit message: un tour c'est 2pi

File: tools/xacro/asterix.xacro (robot description, xacro)
@@ -90,5 +90,5 @@
     <parent link="robotbase"/>
     <child link="sensor_back_left"/>
-    <origin xyz="-0.096 0.1 0.05" rpy="0 0 1.57"/>
+    <origin xyz="-0.096 0.1 0.05" rpy="0 0 3.14159"/>
   </joint>
   <link name="sensor_back_left">
@@ -104,5 +104,5 @@
     <parent link="robotbase"/>
     <child link="sensor_back_right"/>
-    <origin xyz="-0.096 -0.1 0.05" rpy="0 0 1.57"/>
+    <origin xyz="-0.096 -0.1 0.05" rpy="0 0 3.14159"/>
   </joint>
   <link name="sensor_back_right">

Commit message: Formatting + prefix

File: tools/xacro/asterix.xacro (robot description, xacro)
@@ -3,11 +3,12 @@
   <xacro:include filename="colors.xacro"/>
   <xacro:include filename="inertias.xacro"/>
-  <link name="base_link"/>
-  <joint name="base_joint" type="fixed">
-    <parent link="base_link"/>
-    <child link="robotbase"/>
+  <xacro:arg name="tf_prefix" default=""/>
+  <link name="$(arg tf_prefix)base_link"/>
+  <joint name="$(arg tf_prefix)base_joint" type="fixed">
+    <parent link="$(arg tf_prefix)base_link"/>
+    <child link="$(arg tf_prefix)robotbase"/>
     <origin xyz="0.0 0.0 0.16" rpy="0 0 0"/>
   </joint>
-  <link name="robotbase">
+  <link name="$(arg tf_prefix)robotbase">
     <xacro:box_inertia m="4" w="0.2" h="0.26" d="0.32"/>
     <visual>
@@ -20,17 +21,17 @@
     <collision>
       <origin xyz="0.0 0.0 0.0" rpy="0.0 0.0 0.0"/>
-        <geometry>
-          <box size="0.25 0.30 0.35"/>
-        </geometry>
+      <geometry>
+        <box size="0.25 0.30 0.35"/>
+      </geometry>
     </collision>
   </link>
-  <joint name="wheel_left_joint" type="continuous">
-    <parent link="robotbase"/>
-    <child link="wheel_left_link"/>
+  <joint name="$(arg tf_prefix)wheel_left_joint" type="continuous">
+    <parent link="$(arg tf_prefix)robotbase"/>
+    <child link="$(arg tf_prefix)wheel_left_link"/>
     <origin xyz="0.0 0.13 -0.13" rpy="0 0 0"/>
     <axis xyz="0 1 0"/>
     <dynamics damping="0.7"/>
   </joint>
-  <link name="wheel_left_link">
+  <link name="$(arg tf_prefix)wheel_left_link">
     <xacro:cylinder_inertia m="0.2" r="0.04" h="0.01"/>
     <visual>
@@ -42,12 +43,12 @@
     </visual>
   </link>
-  <joint name="wheel_right_joint" type="continuous">
-    <parent link="robotbase"/>
-    <child link="wheel_right_link"/>
+  <joint name="$(arg tf_prefix)wheel_right_joint" type="continuous">
+    <parent link="$(arg tf_prefix)robotbase"/>
+    <child link="$(arg tf_prefix)wheel_right_link"/>
     <origin xyz="0.0 -0.13 -0.13" rpy="0 0 0"/>
     <axis xyz="0 1 0"/>
     <dynamics damping="0.7"/>
   </joint>
-  <link name="wheel_right_link">
+  <link name="$(arg tf_prefix)wheel_right_link">
     <xacro:cylinder_inertia m="0.2" r="0.04" h="0.01"/>
     <visual>
@@ -59,10 +60,10 @@
     </visual>
   </link>
-  <joint name="sensor_front_left_joint" type="fixed">
-    <parent link="robotbase"/>
-    <child link="sensor_front_left"/>
+  <joint name="$(arg tf_prefix)sensor_front_left_joint" type="fixed">
+    <parent link="$(arg tf_prefix)robotbase"/>
+    <child link="$(arg tf_prefix)sensor_front_left"/>
     <origin xyz="0.096 0.1 0.05" rpy="0 0 0"/>
   </joint>
-  <link name="sensor_front_left">
+  <link name="$(arg tf_prefix)sensor_front_left">
     <visual>
       <origin xyz="0 0 0" rpy="0 0 0"/>
@@ -73,10 +74,10 @@
     </visual>
   </link>
-  <joint name="sensor_front_right_joint" type="fixed">
-    <parent link="robotbase"/>
-    <child link="sensor_front_right"/>
+  <joint name="$(arg tf_prefix)sensor_front_right_joint" type="fixed">
+    <parent link="$(arg tf_prefix)robotbase"/>
+    <child link="$(arg tf_prefix)sensor_front_right"/>
     <origin xyz="0.096 -0.1 0.05" rpy="0 0 0"/>
   </joint>
-  <link name="sensor_front_right">
+  <link name="$(arg tf_prefix)sensor_front_right">
     <visual>
       <origin xyz="0 0 0" rpy="0 0 0"/>
@@ -87,10 +88,9 @@
     </visual>
   </link>
-  <joint name="sensor_back_left_joint" type="fixed">
-    <parent link="robotbase"/>
-    <child link="sensor_back_left"/>
-    <origin xyz="-0.096 0.1 0.05" rpy="0 0 3.14159"/>
+  <joint name="$(arg tf_prefix)sensor_back_left_joint" type="fixed">
+    <parent link="$(arg tf_prefix)robotbase"/>
+    <child link="$(arg tf_prefix)sensor_back_left"/>
   </joint>
-  <link name="sensor_back_left">
+  <link name="$(arg tf_prefix)sensor_back_left">
     <visual>
       <origin xyz="0 0 0" rpy="0 0 0"/>
@@ -101,10 +101,10 @@
     </visual>
   </link>
-  <joint name="sensor_back_right_joint" type="fixed">
-    <parent link="robotbase"/>
-    <child link="sensor_back_right"/>
+  <joint name="$(arg tf_prefix)sensor_back_right_joint" type="fixed">
+    <parent link="$(arg tf_prefix)robotbase"/>
+    <child link="$(arg tf_prefix)sensor_back_right"/>
     <origin xyz="-0.096 -0.1 0.05" rpy="0 0 3.14159"/>
   </joint>
-  <link name="sensor_back_right">
+  <link name="$(arg tf_prefix)sensor_back_right">
     <visual>
       <origin xyz="0 0 0" rpy="0 0 0"/>

File: tools/xacro/colors.xacro (robot description, xacro)
@@ -2,5 +2,5 @@
 <robot>
   <material name="black">
-      <color rgba="0.0 0.0 0.0 1.0"/>
+    <color rgba="0.0 0.0 0.0 1.0"/>
   </material>
   <material name="dark">

File: tools/xacro/inertias.xacro (robot description, xacro)
@@ -1,22 +1,22 @@
 <?xml version="1.0" ?>
 <robot xmlns:xacro="http://www.ros.org/wiki/xacro">
-<!--Interial macros-->
-<xacro:macro name="cylinder_inertia" params="m r h">
-  <inertial>
-    <mass value="${m}"/>
-    <inertia ixx="${m*(3*r*r+h*h)/12}" ixy = "0" ixz = "0" iyy="${m*(3*r*r+h*h)/12}" iyz = "0" izz="${m*r*r/2}"/>
-  </inertial>
-</xacro:macro>
-<xacro:macro name="box_inertia" params="m w h d">
-  <inertial>
-    <mass value="${m}"/>
-    <inertia ixx="${m / 12.0 * (d*d + h*h)}" ixy="0.0" ixz="0.0" iyy="${m / 12.0 * (w*w + h*h)}" iyz="0.0" izz="${m / 12.0 * (w*w + d*d)}"/>
-  </inertial>
-</xacro:macro>
-<xacro:macro name="sphere_inertia" params="m r">
-  <inertial>
-    <mass value="${m}"/>
-    <inertia ixx="${2.0*m*(r*r)/5.0}" ixy="0.0" ixz="0.0" iyy="${2.0*m*(r*r)/5.0}" iyz="0.0" izz="${2.0*m*(r*r)/5.0}"/>
-  </inertial>
-</xacro:macro>
+  <!--Interial macros-->
+  <xacro:macro name="cylinder_inertia" params="m r h">
+    <inertial>
+      <mass value="${m}"/>
+      <inertia ixx="${m*(3*r*r+h*h)/12}" ixy="0" ixz="0" iyy="${m*(3*r*r+h*h)/12}" iyz="0" izz="${m*r*r/2}"/>
+    </inertial>
+  </xacro:macro>
+  <xacro:macro name="box_inertia" params="m w h d">
+    <inertial>
+      <mass value="${m}"/>
+      <inertia ixx="${m / 12.0 * (d*d + h*h)}" ixy="0.0" ixz="0.0" iyy="${m / 12.0 * (w*w + h*h)}" iyz="0.0" izz="${m / 12.0 * (w*w + d*d)}"/>
+    </inertial>
+  </xacro:macro>
+  <xacro:macro name="sphere_inertia" params="m r">
+    <inertial>
+      <mass value="${m}"/>
+      <inertia ixx="${2.0*m*(r*r)/5.0}" ixy="0.0" ixz="0.0" iyy="${2.0*m*(r*r)/5.0}" iyz="0.0" izz="${2.0*m*(r*r)/5.0}"/>
+    </inertial>
+  </xacro:macro>
 </robot>

Commit message: Added some templating

File: tools/xacro/asterix.xacro (robot description, xacro)
@@ -1,117 +1,7 @@
 <?xml version="1.0" ?>
-<robot name="asterix" xmlns:xacro="http://www.ros.org/wiki/xacro">
-  <xacro:include filename="colors.xacro"/>
-  <xacro:include filename="inertias.xacro"/>
-  <xacro:arg name="tf_prefix" default=""/>
-  <link name="$(arg tf_prefix)base_link"/>
-  <joint name="$(arg tf_prefix)base_joint" type="fixed">
-    <parent link="$(arg tf_prefix)base_link"/>
-    <child link="$(arg tf_prefix)robotbase"/>
-    <origin xyz="0.0 0.0 0.16" rpy="0 0 0"/>
-  </joint>
-  <link name="$(arg tf_prefix)robotbase">
-    <xacro:box_inertia m="4" w="0.2" h="0.26" d="0.32"/>
-    <visual>
-      <origin xyz="0.0 0.0 0.0" rpy="0.0 0.0 0.0"/>
-      <geometry>
-        <box size="0.2 0.26 0.32"/>
-      </geometry>
-      <material name="blue"/>
-    </visual>
-    <collision>
-      <origin xyz="0.0 0.0 0.0" rpy="0.0 0.0 0.0"/>
-      <geometry>
-        <box size="0.25 0.30 0.35"/>
-      </geometry>
-    </collision>
-  </link>
-  <joint name="$(arg tf_prefix)wheel_left_joint" type="continuous">
-    <parent link="$(arg tf_prefix)robotbase"/>
-    <child link="$(arg tf_prefix)wheel_left_link"/>
-    <origin xyz="0.0 0.13 -0.13" rpy="0 0 0"/>
-    <axis xyz="0 1 0"/>
-    <dynamics damping="0.7"/>
-  </joint>
-  <link name="$(arg tf_prefix)wheel_left_link">
-    <xacro:cylinder_inertia m="0.2" r="0.04" h="0.01"/>
-    <visual>
-      <origin xyz="0 0 0" rpy="1.57 0 0"/>
-      <geometry>
-        <cylinder length="0.01" radius="0.04"/>
-      </geometry>
-      <material name="dark"/>
-    </visual>
-  </link>
-  <joint name="$(arg tf_prefix)wheel_right_joint" type="continuous">
-    <parent link="$(arg tf_prefix)robotbase"/>
-    <child link="$(arg tf_prefix)wheel_right_link"/>
-    <origin xyz="0.0 -0.13 -0.13" rpy="0 0 0"/>
-    <axis xyz="0 1 0"/>
-    <dynamics damping="0.7"/>
-  </joint>
-  <link name="$(arg tf_prefix)wheel_right_link">
-    <xacro:cylinder_inertia m="0.2" r="0.04" h="0.01"/>
-    <visual>
-      <origin xyz="0 0 0" rpy="1.57 0 0"/>
-      <geometry>
-        <cylinder length="0.01" radius="0.04"/>
-      </geometry>
-      <material name="dark"/>
-    </visual>
-  </link>
-  <joint name="$(arg tf_prefix)sensor_front_left_joint" type="fixed">
-    <parent link="$(arg tf_prefix)robotbase"/>
-    <child link="$(arg tf_prefix)sensor_front_left"/>
-    <origin xyz="0.096 0.1 0.05" rpy="0 0 0"/>
-  </joint>
-  <link name="$(arg tf_prefix)sensor_front_left">
-    <visual>
-      <origin xyz="0 0 0" rpy="0 0 0"/>
-      <geometry>
-        <box size="0.01 0.05 0.02"/>
-      </geometry>
-      <material name="white"/>
-    </visual>
-  </link>
-  <joint name="$(arg tf_prefix)sensor_front_right_joint" type="fixed">
-    <parent link="$(arg tf_prefix)robotbase"/>
-    <child link="$(arg tf_prefix)sensor_front_right"/>
-    <origin xyz="0.096 -0.1 0.05" rpy="0 0 0"/>
-  </joint>
-  <link name="$(arg tf_prefix)sensor_front_right">
-    <visual>
-      <origin xyz="0 0 0" rpy="0 0 0"/>
-      <geometry>
-        <box size="0.01 0.05 0.02"/>
-      </geometry>
-      <material name="white"/>
-    </visual>
-  </link>
-  <joint name="$(arg tf_prefix)sensor_back_left_joint" type="fixed">
-    <parent link="$(arg tf_prefix)robotbase"/>
-    <child link="$(arg tf_prefix)sensor_back_left"/>
-  </joint>
-  <link name="$(arg tf_prefix)sensor_back_left">
-    <visual>
-      <origin xyz="0 0 0" rpy="0 0 0"/>
-      <geometry>
-        <box size="0.01 0.05 0.02"/>
-      </geometry>
-      <material name="white"/>
-    </visual>
-  </link>
-  <joint name="$(arg tf_prefix)sensor_back_right_joint" type="fixed">
-    <parent link="$(arg tf_prefix)robotbase"/>
-    <child link="$(arg tf_prefix)sensor_back_right"/>
-    <origin xyz="-0.096 -0.1 0.05" rpy="0 0 3.14159"/>
-  </joint>
-  <link name="$(arg tf_prefix)sensor_back_right">
-    <visual>
-      <origin xyz="0 0 0" rpy="0 0 0"/>
-      <geometry>
-        <box size="0.01 0.05 0.02"/>
-      </geometry>
-      <material name="white"/>
-    </visual>
-  </link>
+<robot name="$(arg robot)" xmlns:xacro="http://www.ros.org/wiki/xacro">
+  <xacro:property name="robotbase_lenght" value="0.2" />
+  <xacro:property name="robotbase_width" value="0.26" />
+  <xacro:property name="robotbase_height" value="0.32" />
+  <xacro:include filename="robot.xacro"/>
 </robot>

Commit message: Asterix & Obelix

File: tools/xacro/asterix.xacro (robot description, xacro)
@@ -1,7 +1,8 @@
 <?xml version="1.0" ?>
-<robot name="$(arg robot)" xmlns:xacro="http://www.ros.org/wiki/xacro">
-  <xacro:property name="robotbase_lenght" value="0.2" />
-  <xacro:property name="robotbase_width" value="0.26" />
-  <xacro:property name="robotbase_height" value="0.32" />
+<robot name="asterix" xmlns:xacro="http://www.ros.org/wiki/xacro">
+  <xacro:property name="robot" value="asterix"/>
+  <xacro:property name="robotbase_lenght" value="0.2"/>
+  <xacro:property name="robotbase_width" value="0.26"/>
+  <xacro:property name="robotbase_height" value="0.32"/>
   <xacro:include filename="robot.xacro"/>
 </robot>

File: tools/xacro/obelix.xacro (robot description, xacro)
@@ -1,4 +1,8 @@
 <?xml version="1.0" ?>
-<robot name="$(arg robot)" xmlns:xacro="http://www.ros.org/wiki/xacro">
+<robot name="obelix" xmlns:xacro="http://www.ros.org/wiki/xacro">
+  <xacro:property name="robot" value="obelix"/>
+  <xacro:property name="robotbase_lenght" value="0.2"/>
+  <xacro:property name="robotbase_width" value="0.26"/>
+  <xacro:property name="robotbase_height" value="0.32"/>
   <xacro:include filename="robot.xacro"/>
 </robot>

File: tools/xacro/robot.xacro (robot description, xacro)
@@ -1,6 +1,5 @@
 <?xml version="1.0" ?>
-<robot name="$(arg robot)" xmlns:xacro="http://www.ros.org/wiki/xacro">
-  <xacro:arg name="robot" default="robot"/>
-  <xacro:arg name="tf_prefix" default="$(arg robot)/"/>
+<robot name="${robot}" xmlns:xacro="http://www.ros.org/wiki/xacro">
+  <xacro:arg name="tf_prefix" default="${robot}/"/>
   <xacro:include filename="colors.xacro"/>
   <xacro:include filename="inertias.xacro"/>

Commit message: Updated dimensions

File: tools/xacro/asterix.xacro (robot description, xacro)
@@ -2,7 +2,9 @@
 <robot name="asterix" xmlns:xacro="http://www.ros.org/wiki/xacro">
   <xacro:property name="robot" value="asterix"/>
-  <xacro:property name="robotbase_lenght" value="0.2"/>
-  <xacro:property name="robotbase_width" value="0.26"/>
+  <xacro:property name="robotbase_lenght" value="0.18"/>
+  <xacro:property name="robotbase_width" value="0.315"/>
   <xacro:property name="robotbase_height" value="0.32"/>
+  <xacro:property name="wheel_radius" value=".0615"/>
+  <xacro:property name="wheel_width" value=".02"/>
   <xacro:include filename="robot.xacro"/>
 </robot>

File: tools/xacro/obelix.xacro (robot description, xacro)
@@ -5,4 +5,6 @@
   <xacro:property name="robotbase_width" value="0.26"/>
   <xacro:property name="robotbase_height" value="0.32"/>
+  <xacro:property name="wheel_radius" value=".04"/>
+  <xacro:property name="wheel_width" value=".01"/>
   <xacro:include filename="robot.xacro"/>
 </robot>

File: tools/xacro/robot.xacro (robot description, xacro)
@@ -34,9 +34,9 @@
   </joint>
   <link name="$(arg tf_prefix)wheel_left_link">
-    <xacro:cylinder_inertia m="0.2" r="0.04" h="0.01"/>
+    <xacro:cylinder_inertia m="0.2" r="${wheel_radius}" h="${wheel_width}"/>
     <visual>
       <origin xyz="0 0 0" rpy="1.57 0 0"/>
       <geometry>
-        <cylinder length="0.01" radius="0.04"/>
+        <cylinder length="${wheel_width}" radius="${wheel_radius}"/>
       </geometry>
       <material name="dark"/>
@@ -51,9 +51,9 @@
   </joint>
   <link name="$(arg tf_prefix)wheel_right_link">
-    <xacro:cylinder_inertia m="0.2" r="0.04" h="0.01"/>
+    <xacro:cylinder_inertia m="0.2" r="${wheel_radius}" h="${wheel_width}"/>
     <visual>
       <origin xyz="0 0 0" rpy="1.57 0 0"/>
       <geometry>
-        <cylinder length="0.01" radius="0.04"/>
+        <cylinder length="${wheel_width}" radius="${wheel_radius}"/>
       </geometry>
       <material name="dark"/>

Commit message: Fix robot URDFs 🤖

File: tools/xacro/asterix.xacro (robot description, xacro)
@@ -1,10 +1,10 @@
 <?xml version="1.0" ?>
 <robot name="asterix" xmlns:xacro="http://www.ros.org/wiki/xacro">
-  <xacro:property name="robot" value="asterix"/>
-  <xacro:property name="robotbase_lenght" value="0.18"/>
-  <xacro:property name="robotbase_width" value="0.315"/>
+  <xacro:property name="robot" value="obelix"/>
+  <xacro:property name="robotbase_lenght" value="0.2"/>
+  <xacro:property name="robotbase_width" value="0.26"/>
   <xacro:property name="robotbase_height" value="0.32"/>
-  <xacro:property name="wheel_radius" value=".0615"/>
-  <xacro:property name="wheel_width" value=".02"/>
+  <xacro:property name="wheel_radius" value=".04"/>
+  <xacro:property name="wheel_width" value=".01"/>
   <xacro:include filename="robot.xacro"/>
 </robot>

File: tools/xacro/obelix.xacro (robot description, xacro)
@@ -1,10 +1,10 @@
 <?xml version="1.0" ?>
 <robot name="obelix" xmlns:xacro="http://www.ros.org/wiki/xacro">
-  <xacro:property name="robot" value="obelix"/>
-  <xacro:property name="robotbase_lenght" value="0.2"/>
-  <xacro:property name="robotbase_width" value="0.26"/>
+  <xacro:property name="robot" value="asterix"/>
+  <xacro:property name="robotbase_lenght" value="0.18"/>
+  <xacro:property name="robotbase_width" value="0.315"/>
   <xacro:property name="robotbase_height" value="0.32"/>
-  <xacro:property name="wheel_radius" value=".04"/>
-  <xacro:property name="wheel_width" value=".01"/>
+  <xacro:property name="wheel_radius" value=".0615"/>
+  <xacro:property name="wheel_width" value=".02"/>
   <xacro:include filename="robot.xacro"/>
 </robot>

Commit message: Fix URDFs

File: tools/xacro/asterix.xacro (robot description, xacro)
@@ -1,5 +1,5 @@
 <?xml version="1.0" ?>
 <robot name="asterix" xmlns:xacro="http://www.ros.org/wiki/xacro">
-  <xacro:property name="robot" value="obelix"/>
+  <xacro:property name="robot" value="asterix"/>
   <xacro:property name="robotbase_lenght" value="0.2"/>
   <xacro:property name="robotbase_width" value="0.26"/>

File: tools/xacro/obelix.xacro (robot description, xacro)
@@ -1,5 +1,5 @@
 <?xml version="1.0" ?>
 <robot name="obelix" xmlns:xacro="http://www.ros.org/wiki/xacro">
-  <xacro:property name="robot" value="asterix"/>
+  <xacro:property name="robot" value="obelix"/>
   <xacro:property name="robotbase_lenght" value="0.18"/>
   <xacro:property name="robotbase_width" value="0.315"/>

File: tools/xacro/robot.xacro (robot description, xacro)
@@ -1,5 +1,5 @@
 <?xml version="1.0" ?>
 <robot name="${robot}" xmlns:xacro="http://www.ros.org/wiki/xacro">
-  <xacro:property name="tf_prefix" value="${robot}/"/>
+  <xacro:property name="tf_prefix" value=""/>
   <xacro:include filename="colors.xacro"/>
   <xacro:include filename="inertias.xacro"/>

Commit message: Fix typo 🙈

File: tools/xacro/asterix.xacro (robot description, xacro)
@@ -2,5 +2,5 @@
 <robot name="asterix" xmlns:xacro="http://www.ros.org/wiki/xacro">
   <xacro:property name="robot" value="asterix"/>
-  <xacro:property name="robotbase_lenght" value="0.2"/>
+  <xacro:property name="robotbase_length" value="0.2"/>
   <xacro:property name="robotbase_width" value="0.26"/>
   <xacro:property name="robotbase_height" value="0.32"/>

File: tools/xacro/obelix.xacro (robot description, xacro)
@@ -2,5 +2,5 @@
 <robot name="obelix" xmlns:xacro="http://www.ros.org/wiki/xacro">
   <xacro:property name="robot" value="obelix"/>
-  <xacro:property name="robotbase_lenght" value="0.18"/>
+  <xacro:property name="robotbase_length" value="0.18"/>
   <xacro:property name="robotbase_width" value="0.315"/>
   <xacro:property name="robotbase_height" value="0.32"/>

File: tools/xacro/robot.xacro (robot description, xacro)
@@ -12,9 +12,9 @@
   </joint>
   <link name="${tf_prefix}robotbase">
-    <xacro:box_inertia m="4" w="${robotbase_lenght}" h="${robotbase_width}" d="${robotbase_height}"/>
+    <xacro:box_inertia m="4" w="${robotbase_length}" h="${robotbase_width}" d="${robotbase_height}"/>
     <visual>
       <origin xyz="0.0 0.0 0.0" rpy="0.0 0.0 0.0"/>
       <geometry>
-        <box size="${robotbase_lenght} ${robotbase_width} ${robotbase_height}"/>
+        <box size="${robotbase_length} ${robotbase_width} ${robotbase_height}"/>
       </geometry>
       <material name="blue"/>
@@ -23,5 +23,5 @@
       <origin xyz="0.0 0.0 0.0" rpy="0.0 0.0 0.0"/>
       <geometry>
-        <box size="${robotbase_lenght+.05} ${robotbase_width+.05} ${robotbase_height+.05}"/>
+        <box size="${robotbase_length+.05} ${robotbase_width+.05} ${robotbase_height+.05}"/>
       </geometry>
     </collision>
